File: arm.kicad_sch (KiCad schematic)
At the start: 11 parts, among them J13 ARM, SW2 ARM, U8 UCS3205

Commit message: progress update week 6
Parts:
- removed J13: ARM, TerminalBlock_Phoenix:TerminalBlock_Phoenix_MKDS-1,5-2-5.08_1x02_P5.08mm_Horizontal, symbol Connector:Screw_Terminal_01x02
- added J12: ARM, Connector_JST:JST_XH_B2B-XH-A_1x02_P2.50mm_Vertical, symbol Connector_Generic:Conn_01x02
- R21: footprint Resistor_SMD:R_1206_3216Metric -> Resistor_SMD:R_2512_6332Metric
Connections:
- net ARM_E: now also J12.1 (Pin_1)
- net ARM_I: now also J12.2 (Pin_2)
Changed lines of the file:
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@@
       (effects (font (size 1.27 1.27)))
     )
-    (property "Footprint" "Resistor_SMD:R_1206_3216Metric" (at 171.196 102.616 90)
+    (property "Footprint" "Resistor_SMD:R_2512_6332Metric" (at 171.196 102.616 90)
       (effects (font (size 1.27 1.27)) hide)
     )
@@
     )
   )
-  (symbol (lib_id "Connector:Screw_Terminal_01x02") (at 85.09 63.5 0) (mirror y) (unit 1)
-    (in_bom yes) (on_board yes) (dnp no) (fields_autoplaced)
-    (property "Reference" "J13" (at 85.09 57.15 0)
+  (symbol (lib_id "Device:C") (at 88.9 109.22 0) (unit 1)
+    (in_bom yes) (on_board yes) (dnp no) (fields_autoplaced)
+    (property "Reference" "C33" (at 92.71 107.95 0)
+      (effects (font (size 1.27 1.27)) (justify left))
+    )
+    (property "Value" "22u" (at 92.71 110.49 0)
+      (effects (font (size 1.27 1.27)) (justify left))
+    )
+    (property "Footprint" "Capacitor_SMD:C_0603_1608Metric" (at 89.8652 113.03 0)
+      (effects (font (size 1.27 1.27)) hide)
+    )
+    (property "Datasheet" "~" (at 88.9 109.22 0)
+      (effects (font (size 1.27 1.27)) hide)
+    )
+    (pin "1")
+    (pin "2")
+    (instances
+      (project "av2324"
+        (path "/f5bfae7e-37ef-453c-b315-6458aa70054f"
+          (reference "C33") (unit 1)
+        )
+        (path "/f5bfae7e-37ef-453c-b315-6458aa70054f/c186b426-2300-4a0e-af51-012322fef314"
+          (reference "C26") (unit 1)
+        )
+      )
+    )
+  )
+  (symbol (lib_id "Connector_Generic:Conn_01x02") (at 85.09 63.5 0) (mirror y) (unit 1)
+    (in_bom yes) (on_board yes) (dnp no) (fields_autoplaced)
+    (property "Reference" "J12" (at 85.09 57.15 0)
       (effects (font (size 1.27 1.27)))
     )
@@
       (effects (font (size 1.27 1.27)))
     )
-    (property "Footprint" "TerminalBlock_Phoenix:TerminalBlock_Phoenix_MKDS-1,5-2-5.08_1x02_P5.08mm_Horizontal" (at 85.09 63.5 0)
+    (property "Footprint" "Connector_JST:JST_XH_B2B-XH-A_1x02_P2.50mm_Vertical" (at 85.09 63.5 0)
       (effects (font (size 1.27 1.27)) hide)
     )
@@
     (instances
       (project "av2324"
-        (path "/f5bfae7e-37ef-453c-b315-6458aa70054f"
+        (path "/f5bfae7e-37ef-453c-b315-6458aa70054f/32ae0883-da14-4189-aed1-7d6ebb961713"
+          (reference "J12") (unit 1)
+        )
+        (path "/f5bfae7e-37ef-453c-b315-6458aa70054f/c186b426-2300-4a0e-af51-012322fef314"
           (reference "J13") (unit 1)
         )
-        (path "/f5bfae7e-37ef-453c-b315-6458aa70054f/c186b426-2300-4a0e-af51-012322fef314"
-          (reference "J13") (unit 1)
-        )
-      )
-    )
-  )
-  (symbol (lib_id "Device:C") (at 88.9 109.22 0) (unit 1)
-    (in_bom yes) (on_board yes) (dnp no) (fields_autoplaced)
-    (property "Reference" "C33" (at 92.71 107.95 0)
-      (effects (font (size 1.27 1.27)) (justify left))
-    )
-    (property "Value" "22u" (at 92.71 110.49 0)
-      (effects (font (size 1.27 1.27)) (justify left))
-    )
-    (property "Footprint" "Capacitor_SMD:C_0603_1608Metric" (at 89.8652 113.03 0)
-      (effects (font (size 1.27 1.27)) hide)
-    )
-    (property "Datasheet" "~" (at 88.9 109.22 0)
-      (effects (font (size 1.27 1.27)) hide)
-    )
-    (pin "1")
-    (pin "2")
-    (instances
-      (project "av2324"
-        (path "/f5bfae7e-37ef-453c-b315-6458aa70054f"
-          (reference "C33") (unit 1)
-        )
-        (path "/f5bfae7e-37ef-453c-b315-6458aa70054f/c186b426-2300-4a0e-af51-012322fef314"
-          (reference "C26") (unit 1)
-        )
-      )
+      )

Commit message: upload before computer reset lol
Parts:
- renumbered C33 to C26, C34 to C27, C35 to C28, J12 to J13, R32 to R10, R21 to R11, R20 to R12, R21 to R13, R19 to R14, SW2 to SW3, U8 to U4
Changed lines of the file:
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@@
   (symbol (lib_id "Device:C") (at 111.76 123.19 0) (unit 1)
     (in_bom yes) (on_board yes) (dnp no) (fields_autoplaced)
-    (property "Reference" "C35" (at 115.57 121.92 0)
+    (property "Reference" "C28" (at 115.57 121.92 0)
       (effects (font (size 1.27 1.27)) (justify left))
     )
@@
     (instances
       (project "av2324"
-        (path "/f5bfae7e-37ef-453c-b315-6458aa70054f"
-          (reference "C35") (unit 1)
-        )
         (path "/f5bfae7e-37ef-453c-b315-6458aa70054f/c186b426-2300-4a0e-af51-012322fef314"
           (reference "C28") (unit 1)
@@
   (symbol (lib_id "Device:R_US") (at 171.45 101.6 270) (unit 1)
     (in_bom yes) (on_board yes) (dnp no) (fields_autoplaced)
-    (property "Reference" "R21" (at 171.45 95.25 90)
+    (property "Reference" "R11" (at 171.45 95.25 90)
       (effects (font (size 1.27 1.27)))
     )
@@
     (instances
       (project "av2324"
-        (path "/f5bfae7e-37ef-453c-b315-6458aa70054f"
-          (reference "R21") (unit 1)
-        )
         (path "/f5bfae7e-37ef-453c-b315-6458aa70054f/c186b426-2300-4a0e-af51-012322fef314"
           (reference "R11") (unit 1)
@@
   (symbol (lib_id "Switch:SW_SPST") (at 100.33 74.93 0) (unit 1)
     (in_bom yes) (on_board yes) (dnp no) (fields_autoplaced)
-    (property "Reference" "SW2" (at 100.33 68.58 0)
+    (property "Reference" "SW3" (at 100.33 68.58 0)
       (effects (font (size 1.27 1.27)))
     )
@@
     (instances
       (project "av2324"
-        (path "/f5bfae7e-37ef-453c-b315-6458aa70054f"
-          (reference "SW2") (unit 1)
-        )
         (path "/f5bfae7e-37ef-453c-b315-6458aa70054f/c186b426-2300-4a0e-af51-012322fef314"
           (reference "SW3") (unit 1)
@@
   (symbol (lib_id "Device:R_US") (at 99.06 123.19 180) (unit 1)
     (in_bom yes) (on_board yes) (dnp no) (fields_autoplaced)
-    (property "Reference" "R19" (at 101.6 121.92 0)
+    (property "Reference" "R14" (at 101.6 121.92 0)
       (effects (font (size 1.27 1.27)) (justify right))
     )
@@
     (instances
       (project "av2324"
-        (path "/f5bfae7e-37ef-453c-b315-6458aa70054f"
-          (reference "R19") (unit 1)
-        )
         (path "/f5bfae7e-37ef-453c-b315-6458aa70054f/c186b426-2300-4a0e-af51-012322fef314"
           (reference "R14") (unit 1)
@@
   (symbol (lib_id "erlib:UCS3205") (at 128.27 109.22 0) (unit 1)
     (in_bom yes) (on_board yes) (dnp no) (fields_autoplaced)
-    (property "Reference" "U8" (at 128.27 93.98 0)
+    (property "Reference" "U4" (at 128.27 93.98 0)
       (effects (font (size 1.27 1.27)))
     )
@@
     (instances
       (project "av2324"
-        (path "/f5bfae7e-37ef-453c-b315-6458aa70054f"
-          (reference "U8") (unit 1)
-        )
         (path "/f5bfae7e-37ef-453c-b315-6458aa70054f/c186b426-2300-4a0e-af51-012322fef314"
           (reference "U4") (unit 1)
@@
   (symbol (lib_id "Device:C") (at 165.1 109.22 0) (unit 1)
     (in_bom yes) (on_board yes) (dnp no) (fields_autoplaced)
-    (property "Reference" "C34" (at 168.91 107.95 0)
+    (property "Reference" "C27" (at 168.91 107.95 0)
       (effects (font (size 1.27 1.27)) (justify left))
     )
@@
     (instances
       (project "av2324"
-        (path "/f5bfae7e-37ef-453c-b315-6458aa70054f"
-          (reference "C34") (unit 1)
-        )
         (path "/f5bfae7e-37ef-453c-b315-6458aa70054f/c186b426-2300-4a0e-af51-012322fef314"
           (reference "C27") (unit 1)
@@
   (symbol (lib_id "Device:R_US") (at 128.27 88.9 90) (unit 1)
     (in_bom yes) (on_board yes) (dnp no) (fields_autoplaced)
-    (property "Reference" "R32" (at 128.27 82.55 90)
+    (property "Reference" "R10" (at 128.27 82.55 90)
       (effects (font (size 1.27 1.27)))
     )
@@
     (instances
       (project "av2324"
-        (path "/f5bfae7e-37ef-453c-b315-6458aa70054f"
-          (reference "R32") (unit 1)
-        )
         (path "/f5bfae7e-37ef-453c-b315-6458aa70054f/c186b426-2300-4a0e-af51-012322fef314"
           (reference "R10") (unit 1)
@@
   (symbol (lib_id "Device:C") (at 88.9 109.22 0) (unit 1)
     (in_bom yes) (on_board yes) (dnp no) (fields_autoplaced)
-    (property "Reference" "C33" (at 92.71 107.95 0)
+    (property "Reference" "C26" (at 92.71 107.95 0)
       (effects (font (size 1.27 1.27)) (justify left))
     )
@@
     (instances
       (project "av2324"
-        (path "/f5bfae7e-37ef-453c-b315-6458aa70054f"
-          (reference "C33") (unit 1)
-        )
         (path "/f5bfae7e-37ef-453c-b315-6458aa70054f/c186b426-2300-4a0e-af51-012322fef314"
           (reference "C26") (unit 1)
@@
   (symbol (lib_id "Connector_Generic:Conn_01x02") (at 85.09 63.5 0) (mirror y) (unit 1)
     (in_bom yes) (on_board yes) (dnp no) (fields_autoplaced)
-    (property "Reference" "J12" (at 85.09 57.15 0)
+    (property "Reference" "J13" (at 85.09 57.15 0)
       (effects (font (size 1.27 1.27)))
     )
@@
     (instances
       (project "av2324"
-        (path "/f5bfae7e-37ef-453c-b315-6458aa70054f/32ae0883-da14-4189-aed1-7d6ebb961713"
-          (reference "J12") (unit 1)
-        )
         (path "/f5bfae7e-37ef-453c-b315-6458aa70054f/c186b426-2300-4a0e-af51-012322fef314"
           (reference "J13") (unit 1)
@@
   (symbol (lib_id "Device:R_US") (at 105.41 109.22 270) (unit 1)
     (in_bom yes) (on_board yes) (dnp no)
-    (property "Reference" "R20" (at 105.41 104.14 90)
+    (property "Reference" "R12" (at 105.41 104.14 90)
       (effects (font (size 1.27 1.27)))
     )
@@
     (instances
       (project "av2324"
-        (path "/f5bfae7e-37ef-453c-b315-6458aa70054f"
-          (reference "R20") (unit 1)
-        )
         (path "/f5bfae7e-37ef-453c-b315-6458aa70054f/c186b426-2300-4a0e-af51-012322fef314"
           (reference "R12") (unit 1)
@@
   (symbol (lib_id "Device:R_US") (at 153.67 110.49 180) (unit 1)
     (in_bom yes) (on_board yes) (dnp no) (fields_autoplaced)
-    (property "Reference" "R21" (at 156.21 109.22 0)
+    (property "Reference" "R13" (at 156.21 109.22 0)
       (effects (font (size 1.27 1.27)) (justify right))
     )
@@
     (instances
       (project "av2324"
-        (path "/f5bfae7e-37ef-453c-b315-6458aa70054f"
-          (reference "R21") (unit 1)
-        )
         (path "/f5bfae7e-37ef-453c-b315-6458aa70054f/c186b426-2300-4a0e-af51-012322fef314"
           (reference "R13") (unit 1)
