File: av2324.kicad_sch (KiCad schematic)
At the start: 43 parts, among them J1 USB, J10 Conn_01x03, J11 Conn_01x03, J2 BATT, J3 Conn_01x03, J4 Conn_01x03, J5 RADIO, J6 SERIAL, J7 EXT, J8 Conn_01x03, J9 Conn_01x03, SW1 RESET, U1 ATSAMD51J20A-M, Y1 12MHz

Commit message: progress update week 6
Parts:
- added R35: 1k, Resistor_SMD:R_0603_1608Metric, symbol Device:R_US
- added R36: 330, Resistor_SMD:R_0603_1608Metric, symbol Device:R_US
- C1, C3: value Cl -> 18p
Connections:
- net +3.3V: now also R35.2
- net SWCLK: now also R35.1
- net ~{RESET}: now also R36.2; no longer SW1.2
- new net: R36.1, SW1.2
Other:
- moved on the sheet: C2, SW1
Changed lines of the file:
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@@
     (stroke (width 0) (type default))
   )
-  (wire (pts (xy 228.6 25.4) (xy 215.9 25.4))
+  (wire (pts (xy 228.6 25.4) (xy 226.06 25.4))
     (stroke (width 0) (type default))
   )
@@
     (stroke (width 0) (type default))
   )
+  (wire (pts (xy 215.9 25.4) (xy 215.9 27.94))
+    (stroke (width 0) (type default))
+  )
   (wire (pts (xy 215.9 86.36) (xy 203.2 86.36))
     (stroke (width 0) (type default))
@@
     (stroke (width 0) (type default))
   )
-  (wire (pts (xy 215.9 36.83) (xy 215.9 38.1))
-    (stroke (width 0) (type default))
-  )
   (wire (pts (xy 152.4 91.44) (xy 165.1 91.44))
     (stroke (width 0) (type default))
@@
     (stroke (width 0) (type default))
   )
+  (wire (pts (xy 218.44 25.4) (xy 215.9 25.4))
+    (stroke (width 0) (type default))
+  )
   (wire (pts (xy 228.6 142.24) (xy 236.22 142.24))
     (stroke (width 0) (type default))
@@
     (stroke (width 0) (type default))
   )
-  (wire (pts (xy 215.9 25.4) (xy 215.9 26.67))
-    (stroke (width 0) (type default))
-  )
-  (wire (pts (xy 228.6 35.56) (xy 228.6 38.1))
+  (wire (pts (xy 320.04 187.96) (xy 320.04 190.5))
     (stroke (width 0) (type default))
   )
-  (wire (pts (xy 320.04 187.96) (xy 320.04 190.5))
+  (wire (pts (xy 215.9 121.92) (xy 215.9 124.46))
     (stroke (width 0) (type default))
   )
@@
     (stroke (width 0) (type default))
   )
+  (wire (pts (xy 228.6 36.83) (xy 228.6 38.1))
+    (stroke (width 0) (type default))
+  )
   (wire (pts (xy 203.2 76.2) (xy 215.9 76.2))
     (stroke (width 0) (type default))
@@
     (stroke (width 0) (type default))
   )
+  (wire (pts (xy 215.9 132.08) (xy 215.9 134.62))
+    (stroke (width 0) (type default))
+  )
   (wire (pts (xy 127 152.4) (xy 127 154.94))
     (stroke (width 0) (type default))
@@
     (stroke (width 0) (type default))
   )
+  (wire (pts (xy 215.9 134.62) (xy 236.22 134.62))
+    (stroke (width 0) (type default))
+  )
   (wire (pts (xy 271.78 93.98) (xy 279.4 93.98))
     (stroke (width 0) (type default))
@@
     (stroke (width 0) (type default))
   )
-  (wire (pts (xy 228.6 134.62) (xy 236.22 134.62))
-    (stroke (width 0) (type default))
-  )
   (wire (pts (xy 292.1 29.21) (xy 292.1 31.75))
     (stroke (width 0) (type default))
@@
     (stroke (width 0) (type default))
   )
-  (wire (pts (xy 228.6 27.94) (xy 228.6 25.4))
-    (stroke (width 0) (type default))
-  )
   (wire (pts (xy 166.37 31.75) (xy 166.37 40.64))
     (stroke (width 0) (type default))
@@
     (stroke (width 0) (type default))
   )
+  (wire (pts (xy 228.6 26.67) (xy 228.6 25.4))
+    (stroke (width 0) (type default))
+  )
   (wire (pts (xy 342.9 93.98) (xy 330.2 93.98))
     (stroke (width 0) (type default))
@@
     (stroke (width 0) (type default))
   )
+  (wire (pts (xy 215.9 35.56) (xy 215.9 38.1))
+    (stroke (width 0) (type default))
+  )
   (wire (pts (xy 203.2 78.74) (xy 215.9 78.74))
     (stroke (width 0) (type default))
@@
     )
   )
+  (symbol (lib_id "Device:R_US") (at 222.25 25.4 270) (unit 1)
+    (in_bom yes) (on_board yes) (dnp no) (fields_autoplaced)
+    (property "Reference" "R36" (at 222.25 19.05 90)
+      (effects (font (size 1.27 1.27)))
+    )
+    (property "Value" "330" (at 222.25 21.59 90)
+      (effects (font (size 1.27 1.27)))
+    )
+    (property "Footprint" "Resistor_SMD:R_0603_1608Metric" (at 221.996 26.416 90)
+      (effects (font (size 1.27 1.27)) hide)
+    )
+    (property "Datasheet" "~" (at 222.25 25.4 0)
+      (effects (font (size 1.27 1.27)) hide)
+    )
+    (pin "1")
+    (pin "2")
+    (instances
+      (project "av2324"
+        (path "/f5bfae7e-37ef-453c-b315-6458aa70054f"
+          (reference "R36") (unit 1)
+        )
+        (path "/f5bfae7e-37ef-453c-b315-6458aa70054f/32ae0883-da14-4189-aed1-7d6ebb961713"
+          (reference "R9") (unit 1)
+        )
+      )
+    )
+  )
   (symbol (lib_id "power:GND") (at 391.16 199.39 0) (unit 1)
     (in_bom yes) (on_board yes) (dnp no) (fields_autoplaced)
@@
     )
   )
-  (symbol (lib_id "Switch:SW_Push") (at 215.9 31.75 90) (unit 1)
+  (symbol (lib_id "Switch:SW_Push") (at 228.6 31.75 90) (unit 1)
     (in_bom yes) (on_board yes) (dnp no) (fields_autoplaced)
-    (property "Reference" "SW1" (at 217.17 30.48 90)
+    (property "Reference" "SW1" (at 229.87 30.48 90)
       (effects (font (size 1.27 1.27)) (justify right))
     )
-    (property "Value" "RESET" (at 217.17 33.02 90)
+    (property "Value" "RESET" (at 229.87 33.02 90)
       (effects (font (size 1.27 1.27)) (justify right))
     )
-    (property "Footprint" "Button_Switch_SMD:SW_SPST_PTS810" (at 210.82 31.75 0)
+    (property "Footprint" "Button_Switch_SMD:SW_SPST_PTS810" (at 223.52 31.75 0)
       (effects (font (size 1.27 1.27)) hide)
     )
-    (property "Datasheet" "~" (at 210.82 31.75 0)
+    (property "Datasheet" "~" (at 223.52 31.75 0)
       (effects (font (size 1.27 1.27)) hide)
     )
@@
     )
   )
+  (symbol (lib_id "power:+3.3V") (at 215.9 121.92 0) (unit 1)
+    (in_bom yes) (on_board yes) (dnp no) (fields_autoplaced)
+    (property "Reference" "#PWR071" (at 215.9 125.73 0)
+      (effects (font (size 1.27 1.27)) hide)
+    )
+    (property "Value" "+3.3V" (at 215.9 116.84 0)
+      (effects (font (size 1.27 1.27)))
+    )
+    (property "Footprint" "" (at 215.9 121.92 0)
+      (effects (font (size 1.27 1.27)) hide)
+    )
+    (property "Datasheet" "" (at 215.9 121.92 0)
+      (effects (font (size 1.27 1.27)) hide)
+    )
+    (pin "1")
+    (instances
+      (project "av2324"
+        (path "/f5bfae7e-37ef-453c-b315-6458aa70054f"
+          (reference "#PWR071") (unit 1)
+        )
+      )
+    )
+  )
   (symbol (lib_id "power:+5VP") (at 86.36 152.4 0) (unit 1)
     (in_bom yes) (on_board yes) (dnp no) (fields_autoplaced)
@@
       (effects (font (size 1.27 1.27)))
     )
-    (property "Value" "Cl" (at 185.4263 34.29 90)
+    (property "Value" "18p" (at 185.4263 34.29 90)
       (effects (font (size 1.27 1.27)))
     )
@@
     )
   )
-  (symbol (lib_id "Device:C") (at 228.6 31.75 0) (unit 1)
+  (symbol (lib_id "Device:C") (at 215.9 31.75 0) (unit 1)
     (in_bom yes) (on_board yes) (dnp no) (fields_autoplaced)
-    (property "Reference" "C2" (at 232.41 30.48 0)
+    (property "Reference" "C2" (at 219.71 30.48 0)
       (effects (font (size 1.27 1.27)) (justify left))
     )
-    (property "Value" "0.1u" (at 232.41 33.02 0)
+    (property "Value" "0.1u" (at 219.71 33.02 0)
       (effects (font (size 1.27 1.27)) (justify left))
     )
-    (property "Footprint" "Capacitor_SMD:C_0603_1608Metric" (at 229.5652 35.56 0)
+    (property "Footprint" "Capacitor_SMD:C_0603_1608Metric" (at 216.8652 35.56 0)
       (effects (font (size 1.27 1.27)) hide)
     )
-    (property "Datasheet" "~" (at 228.6 31.75 0)
+    (property "Datasheet" "~" (at 215.9 31.75 0)
       (effects (font (size 1.27 1.27)) hide)
     )
@@
     )
   )
+  (symbol (lib_id "Device:R_US") (at 215.9 128.27 180) (unit 1)
+    (in_bom yes) (on_board yes) (dnp no) (fields_autoplaced)
+    (property "Reference" "R35" (at 218.44 127 0)
+      (effects (font (size 1.27 1.27)) (justify right))
+    )
+    (property "Value" "1k" (at 218.44 129.54 0)
+      (effects (font (size 1.27 1.27)) (justify right))
+    )
+    (property "Footprint" "Resistor_SMD:R_0603_1608Metric" (at 214.884 128.016 90)
+      (effects (font (size 1.27 1.27)) hide)
+    )
+    (property "Datasheet" "~" (at 215.9 128.27 0)
+      (effects (font (size 1.27 1.27)) hide)
+    )
+    (pin "1")
+    (pin "2")
+    (instances
+      (project "av2324"
+        (path "/f5bfae7e-37ef-453c-b315-6458aa70054f"
+          (reference "R35") (unit 1)
+        )
+        (path "/f5bfae7e-37ef-453c-b315-6458aa70054f/32ae0883-da14-4189-aed1-7d6ebb961713"
+          (reference "R9") (unit 1)
+        )
+      )
+    )
+  )
   (symbol (lib_id "Connector_Generic:Conn_01x03") (at 93.98 130.81 0) (unit 1)
     (in_bom yes) (on_board yes) (dnp no) (fields_autoplaced)
@@
       (effects (font (size 1.27 1.27)))
     )
-    (property "Value" "Cl" (at 185.4263 21.59 90)
+    (property "Value" "18p" (at 185.4263 21.59 90)
       (effects (font (size 1.27 1.27)))
     )

Commit message: upload before computer reset lol
Parts:
- added C37: 0.1u, Capacitor_SMD:C_0603_1608Metric, symbol Device:C
- added J19: Micro_SD_Card_Det1, symbol Connector:Micro_SD_Card_Det1
- added R37: 10k, Resistor_SMD:R_0603_1608Metric, symbol Device:R_US
Connections:
- net +3.3V: now also C37.1, J19.4 (VDD), R37.1
- net GND: now also C37.2, J19.10 (SHIELD), J19.6 (VSS)
- net MISO: now also J19.7 (DAT0)
- net MOSI: now also J19.3 (CMD)
- net SCK: now also J19.5 (CLK)
- new net SD~{CS}: J19.2 (DAT3/CD), R37.2
- new net SD~{DET}: J19.9 (DET)
- no-connect marks 4 -> 6
