File: baro.kicad_sch (KiCad schematic)
At the start: 4 parts, among them U6 BMP388

Commit message: upload before computer reset lol
Parts:
- R16: renamed from R9; value 30k -> 10k
- renumbered C25 to C32, C26 to C33
Changed lines of the file:
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@@
     (instances
       (project "av2324"
-        (path "/f5bfae7e-37ef-453c-b315-6458aa70054f"
-          (reference "U6") (unit 1)
-        )
         (path "/f5bfae7e-37ef-453c-b315-6458aa70054f/3dc22ab4-b01a-4be5-83a7-724a49c8c7a4"
           (reference "U6") (unit 1)
@@
   (symbol (lib_id "Device:C") (at 165.1 88.9 0) (unit 1)
     (in_bom yes) (on_board yes) (dnp no) (fields_autoplaced)
-    (property "Reference" "C26" (at 168.91 87.63 0)
+    (property "Reference" "C33" (at 168.91 87.63 0)
       (effects (font (size 1.27 1.27)) (justify left))
     )
@@
     (instances
       (project "av2324"
-        (path "/f5bfae7e-37ef-453c-b315-6458aa70054f"
-          (reference "C26") (unit 1)
-        )
         (path "/f5bfae7e-37ef-453c-b315-6458aa70054f/3dc22ab4-b01a-4be5-83a7-724a49c8c7a4"
           (reference "C33") (unit 1)
@@
   (symbol (lib_id "Device:R_US") (at 114.3 77.47 0) (unit 1)
     (in_bom yes) (on_board yes) (dnp no) (fields_autoplaced)
-    (property "Reference" "R9" (at 116.84 76.2 0)
+    (property "Reference" "R16" (at 116.84 76.2 0)
       (effects (font (size 1.27 1.27)) (justify left))
     )
-    (property "Value" "30k" (at 116.84 78.74 0)
+    (property "Value" "10k" (at 116.84 78.74 0)
       (effects (font (size 1.27 1.27)) (justify left))
     )
@@
     (instances
       (project "av2324"
-        (path "/f5bfae7e-37ef-453c-b315-6458aa70054f"
-          (reference "R9") (unit 1)
-        )
         (path "/f5bfae7e-37ef-453c-b315-6458aa70054f/3dc22ab4-b01a-4be5-83a7-724a49c8c7a4"
           (reference "R16") (unit 1)
@@
   (symbol (lib_id "Device:C") (at 152.4 88.9 0) (unit 1)
     (in_bom yes) (on_board yes) (dnp no) (fields_autoplaced)
-    (property "Reference" "C25" (at 156.21 87.63 0)
+    (property "Reference" "C32" (at 156.21 87.63 0)
       (effects (font (size 1.27 1.27)) (justify left))
     )
@@
     (instances
       (project "av2324"
-        (path "/f5bfae7e-37ef-453c-b315-6458aa70054f"
-          (reference "C25") (unit 1)
-        )
         (path "/f5bfae7e-37ef-453c-b315-6458aa70054f/3dc22ab4-b01a-4be5-83a7-724a49c8c7a4"
           (reference "C32") (unit 1)
