File: flash.kicad_sch (KiCad schematic)
At the start: 3 parts, among them U7 S25FL128LAG

Commit message: upload before computer reset lol
Parts:
- renumbered C27 to C34, R10 to R17
Changed lines of the file:
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@@
   (symbol (lib_id "Device:C") (at 152.4 88.9 0) (unit 1)
     (in_bom yes) (on_board yes) (dnp no) (fields_autoplaced)
-    (property "Reference" "C27" (at 156.21 87.63 0)
+    (property "Reference" "C34" (at 156.21 87.63 0)
       (effects (font (size 1.27 1.27)) (justify left))
     )
@@
     (instances
       (project "av2324"
-        (path "/f5bfae7e-37ef-453c-b315-6458aa70054f"
-          (reference "C27") (unit 1)
-        )
         (path "/f5bfae7e-37ef-453c-b315-6458aa70054f/434c939d-1c96-461b-b517-50373bc7992e"
           (reference "C34") (unit 1)
@@
   (symbol (lib_id "Device:R_US") (at 114.3 74.93 0) (unit 1)
     (in_bom yes) (on_board yes) (dnp no) (fields_autoplaced)
-    (property "Reference" "R10" (at 116.84 73.66 0)
+    (property "Reference" "R17" (at 116.84 73.66 0)
       (effects (font (size 1.27 1.27)) (justify left))
     )
@@
     (instances
       (project "av2324"
-        (path "/f5bfae7e-37ef-453c-b315-6458aa70054f"
-          (reference "R10") (unit 1)
-        )
         (path "/f5bfae7e-37ef-453c-b315-6458aa70054f/434c939d-1c96-461b-b517-50373bc7992e"
           (reference "R17") (unit 1)
@@
     (instances
       (project "av2324"
-        (path "/f5bfae7e-37ef-453c-b315-6458aa70054f"
-          (reference "U7") (unit 1)
-        )
         (path "/f5bfae7e-37ef-453c-b315-6458aa70054f/434c939d-1c96-461b-b517-50373bc7992e"
           (reference "U7") (unit 1)
