File: imu.kicad_sch (KiCad schematic)
At the start: 4 parts, among them U4 LSM6DSO32

Commit message: upload before computer reset lol
Parts:
- renumbered C21 to C35, C22 to C36, R7 to R26, U4 to U8
Changed lines of the file:
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@@
   (symbol (lib_id "Device:R_US") (at 119.38 85.09 0) (unit 1)
     (in_bom yes) (on_board yes) (dnp no) (fields_autoplaced)
-    (property "Reference" "R7" (at 121.92 83.82 0)
+    (property "Reference" "R26" (at 121.92 83.82 0)
       (effects (font (size 1.27 1.27)) (justify left))
     )
@@
     (instances
       (project "av2324"
-        (path "/f5bfae7e-37ef-453c-b315-6458aa70054f"
-          (reference "R7") (unit 1)
-        )
         (path "/f5bfae7e-37ef-453c-b315-6458aa70054f/7bb81c0f-5300-4d5f-9405-667383f80021"
           (reference "R26") (unit 1)
@@
   (symbol (lib_id "Device:C") (at 170.18 102.87 0) (unit 1)
     (in_bom yes) (on_board yes) (dnp no) (fields_autoplaced)
-    (property "Reference" "C22" (at 173.99 101.6 0)
+    (property "Reference" "C36" (at 173.99 101.6 0)
       (effects (font (size 1.27 1.27)) (justify left))
     )
@@
     (instances
       (project "av2324"
-        (path "/f5bfae7e-37ef-453c-b315-6458aa70054f"
-          (reference "C22") (unit 1)
-        )
         (path "/f5bfae7e-37ef-453c-b315-6458aa70054f/7bb81c0f-5300-4d5f-9405-667383f80021"
           (reference "C36") (unit 1)
@@
   (symbol (lib_id "erlib:LSM6DSO32") (at 139.7 101.6 0) (unit 1)
     (in_bom yes) (on_board yes) (dnp no)
-    (property "Reference" "U4" (at 144.78 83.82 0)
+    (property "Reference" "U8" (at 144.78 83.82 0)
       (effects (font (size 1.27 1.27)) (justify left))
     )
@@
     (instances
       (project "av2324"
-        (path "/f5bfae7e-37ef-453c-b315-6458aa70054f"
-          (reference "U4") (unit 1)
-        )
         (path "/f5bfae7e-37ef-453c-b315-6458aa70054f/7bb81c0f-5300-4d5f-9405-667383f80021"
           (reference "U8") (unit 1)
@@
   (symbol (lib_id "Device:C") (at 158.75 102.87 0) (unit 1)
     (in_bom yes) (on_board yes) (dnp no) (fields_autoplaced)
-    (property "Reference" "C21" (at 162.56 101.6 0)
+    (property "Reference" "C35" (at 162.56 101.6 0)
       (effects (font (size 1.27 1.27)) (justify left))
     )
@@
     (instances
       (project "av2324"
-        (path "/f5bfae7e-37ef-453c-b315-6458aa70054f"
-          (reference "C21") (unit 1)
-        )
         (path "/f5bfae7e-37ef-453c-b315-6458aa70054f/7bb81c0f-5300-4d5f-9405-667383f80021"
           (reference "C35") (unit 1)
