File: mag.kicad_sch (KiCad schematic)
At the start: 5 parts, among them U5 LIS3MDL

Commit message: upload before computer reset lol
Parts:
- renumbered C30 to C29, C24 to C30, C23 to C31, R8 to R15
Changed lines of the file:
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@@
   (symbol (lib_id "Device:R_US") (at 124.46 74.93 0) (unit 1)
     (in_bom yes) (on_board yes) (dnp no) (fields_autoplaced)
-    (property "Reference" "R8" (at 127 73.66 0)
+    (property "Reference" "R15" (at 127 73.66 0)
       (effects (font (size 1.27 1.27)) (justify left))
     )
@@
     (instances
       (project "av2324"
-        (path "/f5bfae7e-37ef-453c-b315-6458aa70054f"
-          (reference "R8") (unit 1)
-        )
         (path "/f5bfae7e-37ef-453c-b315-6458aa70054f/8f536043-fe34-459e-b6ce-98bbe2a4e937"
           (reference "R15") (unit 1)
@@
   (symbol (lib_id "Device:C") (at 154.94 97.79 0) (unit 1)
     (in_bom yes) (on_board yes) (dnp no) (fields_autoplaced)
-    (property "Reference" "C30" (at 158.75 96.52 0)
+    (property "Reference" "C29" (at 158.75 96.52 0)
       (effects (font (size 1.27 1.27)) (justify left))
     )
@@
     (instances
       (project "av2324"
-        (path "/f5bfae7e-37ef-453c-b315-6458aa70054f"
-          (reference "C30") (unit 1)
-        )
         (path "/f5bfae7e-37ef-453c-b315-6458aa70054f/8f536043-fe34-459e-b6ce-98bbe2a4e937"
           (reference "C29") (unit 1)
@@
   (symbol (lib_id "Device:C") (at 166.37 97.79 0) (unit 1)
     (in_bom yes) (on_board yes) (dnp no) (fields_autoplaced)
-    (property "Reference" "C24" (at 170.18 96.52 0)
+    (property "Reference" "C30" (at 170.18 96.52 0)
       (effects (font (size 1.27 1.27)) (justify left))
     )
@@
     (instances
       (project "av2324"
-        (path "/f5bfae7e-37ef-453c-b315-6458aa70054f"
-          (reference "C24") (unit 1)
-        )
         (path "/f5bfae7e-37ef-453c-b315-6458aa70054f/8f536043-fe34-459e-b6ce-98bbe2a4e937"
           (reference "C30") (unit 1)
@@
     (instances
       (project "av2324"
-        (path "/f5bfae7e-37ef-453c-b315-6458aa70054f"
-          (reference "U5") (unit 1)
-        )
         (path "/f5bfae7e-37ef-453c-b315-6458aa70054f/8f536043-fe34-459e-b6ce-98bbe2a4e937"
           (reference "U5") (unit 1)
@@
   (symbol (lib_id "Device:C") (at 177.8 97.79 0) (unit 1)
     (in_bom yes) (on_board yes) (dnp no) (fields_autoplaced)
-    (property "Reference" "C23" (at 181.61 96.52 0)
+    (property "Reference" "C31" (at 181.61 96.52 0)
       (effects (font (size 1.27 1.27)) (justify left))
     )
@@
     (instances
       (project "av2324"
-        (path "/f5bfae7e-37ef-453c-b315-6458aa70054f"
-          (reference "C23") (unit 1)
-        )
         (path "/f5bfae7e-37ef-453c-b315-6458aa70054f/8f536043-fe34-459e-b6ce-98bbe2a4e937"
           (reference "C31") (unit 1)
