File: power.kicad_sch (KiCad schematic)
At the start: 26 parts, among them J12 ON, Q1 DMP3098L-7, SW3 ON, U1 TPS565242, U3 AP2112K-3.3

Commit message: progress update week 6
Parts:
- removed J12: ON, TerminalBlock_Phoenix:TerminalBlock_Phoenix_MKDS-1,5-2-5.08_1x02_P5.08mm_Horizontal, symbol Connector:Screw_Terminal_01x02
- added J12: ON, Connector_JST:JST_XH_B2B-XH-A_1x02_P2.50mm_Vertical, symbol Connector_Generic:Conn_01x02
Connections:
- net 5V_EN: now also J12.1 (Pin_1)
- net 5V_UV: now also J12.2 (Pin_2)
Changed lines of the file:
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@@
+    (stroke (width 0) (type default))
+  )
+  (wire (pts (xy 82.55 39.37) (xy 100.33 39.37))
     (stroke (width 0) (type default))
   )
@@
     (stroke (width 0) (type default))
   )
+  (wire (pts (xy 82.55 41.91) (xy 85.09 41.91))
+    (stroke (width 0) (type default))
+  )
   (wire (pts (xy 107.95 127) (xy 119.38 127))
     (stroke (width 0) (type default))
@@
     (stroke (width 0) (type default))
   )
-  (wire (pts (xy 82.55 39.37) (xy 100.33 39.37))
-    (stroke (width 0) (type default))
-  )
   (wire (pts (xy 172.72 101.6) (xy 161.29 101.6))
     (stroke (width 0) (type default))
@@
   )
   (wire (pts (xy 152.4 38.1) (xy 152.4 40.64))
-    (stroke (width 0) (type default))
-  )
-  (wire (pts (xy 82.55 41.91) (xy 85.09 41.91))
     (stroke (width 0) (type default))
   )
@@
         (path "/f5bfae7e-37ef-453c-b315-6458aa70054f/32ae0883-da14-4189-aed1-7d6ebb961713"
           (reference "U3") (unit 1)
+        )
+      )
+    )
+  )
+  (symbol (lib_id "Connector_Generic:Conn_01x02") (at 77.47 39.37 0) (mirror y) (unit 1)
+    (in_bom yes) (on_board yes) (dnp no) (fields_autoplaced)
+    (property "Reference" "J12" (at 77.47 33.02 0)
+      (effects (font (size 1.27 1.27)))
+    )
+    (property "Value" "ON" (at 77.47 35.56 0)
+      (effects (font (size 1.27 1.27)))
+    )
+    (property "Footprint" "Connector_JST:JST_XH_B2B-XH-A_1x02_P2.50mm_Vertical" (at 77.47 39.37 0)
+      (effects (font (size 1.27 1.27)) hide)
+    )
+    (property "Datasheet" "~" (at 77.47 39.37 0)
+      (effects (font (size 1.27 1.27)) hide)
+    )
+    (pin "1")
+    (pin "2")
+    (instances
+      (project "av2324"
+        (path "/f5bfae7e-37ef-453c-b315-6458aa70054f/32ae0883-da14-4189-aed1-7d6ebb961713"
+          (reference "J12") (unit 1)
         )
       )
@@
         )
       )
-    )
-  )
-  (symbol (lib_id "Connector:Screw_Terminal_01x02") (at 77.47 39.37 0) (mirror y) (unit 1)
-    (in_bom yes) (on_board yes) (dnp no) (fields_autoplaced)
-    (property "Reference" "J12" (at 77.47 33.02 0)
-      (effects (font (size 1.27 1.27)))
-    )
-    (property "Value" "ON" (at 77.47 35.56 0)
-      (effects (font (size 1.27 1.27)))
-    )
-    (property "Footprint" "TerminalBlock_Phoenix:TerminalBlock_Phoenix_MKDS-1,5-2-5.08_1x02_P5.08mm_Horizontal" (at 77.47 39.37 0)
-      (effects (font (size 1.27 1.27)) hide)
-    )
-    (property "Datasheet" "~" (at 77.47 39.37 0)
-      (effects (font (size 1.27 1.27)) hide)
-    )
-    (pin "1")
-    (pin "2")
-    (instances
-      (project "av2324"
-        (path "/f5bfae7e-37ef-453c-b315-6458aa70054f"
-          (reference "J12") (unit 1)
-        )
-        (path "/f5bfae7e-37ef-453c-b315-6458aa70054f/32ae0883-da14-4189-aed1-7d6ebb961713"
-          (reference "J12") (unit 1)
-        )
-      )

Commit message: upload before computer reset lol
Parts:
- renumbered C37 to C14, C12 to C15, C13 to C16, C14 to C17, C15 to C18, C16 to C19, C17 to C20, C18 to C21, C29 to C22, C28 to C23, C19 to C24, C20 to C25, D1 to D2, R34 to R3, R35 to R4, R3 to R6, R6 to R7, R4 to R8, R11 to R9, SW3 to SW2, U1 to U2
