File: pyro.kicad_sch (KiCad schematic)
At the start: 6 parts, among them J14 ON, Q2 Q_NMOS_GDS

Commit message: progress update week 6
Parts:
- removed Q2: Q_NMOS_GDS, Package_TO_SOT_SMD:SOT-23, symbol Device:Q_NMOS_GDS
- added Q3: DMN3150L, Package_TO_SOT_SMD:SOT-23, symbol Device:Q_NMOS_GSD
Connections:
- net GND: now also Q3.2 (S)
- net at J14.2 (Pin_2), R34.2: now also Q3.3 (D)
- net at R12.2: now also Q3.1 (G)
Changed lines of the file:
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@@
     (effects (font (size 1.27 1.27)) (justify left))
+  )
+  (symbol (lib_id "Device:Q_NMOS_GSD") (at 127 86.36 90) (mirror x) (unit 1)
+    (in_bom yes) (on_board yes) (dnp no) (fields_autoplaced)
+    (property "Reference" "Q3" (at 127 92.71 90)
+      (effects (font (size 1.27 1.27)))
+    )
+    (property "Value" "DMN3150L" (at 127 95.25 90)
+      (effects (font (size 1.27 1.27)))
+    )
+    (property "Footprint" "Package_TO_SOT_SMD:SOT-23" (at 124.46 91.44 0)
+      (effects (font (size 1.27 1.27)) hide)
+    )
+    (property "Datasheet" "~" (at 127 86.36 0)
+      (effects (font (size 1.27 1.27)) hide)
+    )
+    (pin "1")
+    (pin "2")
+    (pin "3")
+    (instances
+      (project "av2324"
+        (path "/f5bfae7e-37ef-453c-b315-6458aa70054f/0748e7cd-0a3d-4586-8bc7-9a3e9814e06f"
+          (reference "Q3") (unit 1)
+        )
+        (path "/f5bfae7e-37ef-453c-b315-6458aa70054f/2e53005c-227f-416b-8cc3-62e815b93dbf"
+          (reference "Q2") (unit 1)
+        )
+        (path "/f5bfae7e-37ef-453c-b315-6458aa70054f/e82342dd-bc52-4a78-b9b4-ffd05f6fa11a"
+          (reference "Q4") (unit 1)
+        )
+        (path "/f5bfae7e-37ef-453c-b315-6458aa70054f/b2fd81e3-27b1-4390-8a5d-71f8e91885dc"
+          (reference "Q5") (unit 1)
+        )
+      )
+    )
   )
   (symbol (lib_id "Connector:Screw_Terminal_01x02") (at 102.87 86.36 0) (mirror y) (unit 1)
@@
         )
       )
-    )
-  )
-  (symbol (lib_id "Device:Q_NMOS_GDS") (at 127 86.36 270) (unit 1)
-    (in_bom yes) (on_board yes) (dnp no) (fields_autoplaced)
-    (property "Reference" "Q2" (at 127 92.71 90)
-      (effects (font (size 1.27 1.27)))
-    )
-    (property "Value" "Q_NMOS_GDS" (at 127 95.25 90)
-      (effects (font (size 1.27 1.27)))
-    )
-    (property "Footprint" "Package_TO_SOT_SMD:SOT-23" (at 129.54 91.44 0)
-      (effects (font (size 1.27 1.27)) hide)
-    )
-    (property "Datasheet" "~" (at 127 86.36 0)
-      (effects (font (size 1.27 1.27)) hide)
-    )
-    (pin "1")
-    (pin "2")
-    (pin "3")
-    (instances
-      (project "av2324"
-        (path "/f5bfae7e-37ef-453c-b315-6458aa70054f"
-          (reference "Q2") (unit 1)
-        )
-        (path "/f5bfae7e-37ef-453c-b315-6458aa70054f/0748e7cd-0a3d-4586-8bc7-9a3e9814e06f"
-          (reference "Q3") (unit 1)
-        )
-        (path "/f5bfae7e-37ef-453c-b315-6458aa70054f/2e53005c-227f-416b-8cc3-62e815b93dbf"
-          (reference "Q2") (unit 1)
-        )
-        (path "/f5bfae7e-37ef-453c-b315-6458aa70054f/e82342dd-bc52-4a78-b9b4-ffd05f6fa11a"
-          (reference "Q4") (unit 1)
-        )
-        (path "/f5bfae7e-37ef-453c-b315-6458aa70054f/b2fd81e3-27b1-4390-8a5d-71f8e91885dc"
-          (reference "Q5") (unit 1)
-        )
-      )

Commit message: upload before computer reset lol
Parts:
- renumbered J14 to J15, R12 to R22, R34 to R24, R35 to R25
Changed lines of the file:
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@@
   (symbol (lib_id "Connector:Screw_Terminal_01x02") (at 102.87 86.36 0) (mirror y) (unit 1)
     (in_bom yes) (on_board yes) (dnp no) (fields_autoplaced)
-    (property "Reference" "J14" (at 102.87 80.01 0)
+    (property "Reference" "J15" (at 102.87 80.01 0)
       (effects (font (size 1.27 1.27)))
     )
@@
     (instances
       (project "av2324"
-        (path "/f5bfae7e-37ef-453c-b315-6458aa70054f"
-          (reference "J14") (unit 1)
-        )
         (path "/f5bfae7e-37ef-453c-b315-6458aa70054f/0748e7cd-0a3d-4586-8bc7-9a3e9814e06f"
           (reference "J15") (unit 1)
@@
   (symbol (lib_id "Device:R_US") (at 110.49 95.25 180) (unit 1)
     (in_bom yes) (on_board yes) (dnp no) (fields_autoplaced)
-    (property "Reference" "R34" (at 113.03 93.98 0)
+    (property "Reference" "R24" (at 113.03 93.98 0)
       (effects (font (size 1.27 1.27)) (justify right))
     )
@@
     (instances
       (project "av2324"
-        (path "/f5bfae7e-37ef-453c-b315-6458aa70054f"
-          (reference "R34") (unit 1)
-        )
-        (path "/f5bfae7e-37ef-453c-b315-6458aa70054f/32ae0883-da14-4189-aed1-7d6ebb961713"
-          (reference "R34") (unit 1)
-        )
         (path "/f5bfae7e-37ef-453c-b315-6458aa70054f/0748e7cd-0a3d-4586-8bc7-9a3e9814e06f"
           (reference "R24") (unit 1)
@@
     (instances
       (project "av2324"
-        (path "/f5bfae7e-37ef-453c-b315-6458aa70054f"
-          (reference "R23") (unit 1)
-        )
         (path "/f5bfae7e-37ef-453c-b315-6458aa70054f/0748e7cd-0a3d-4586-8bc7-9a3e9814e06f"
           (reference "R23") (unit 1)
@@
   (symbol (lib_id "Device:R_US") (at 110.49 107.95 180) (unit 1)
     (in_bom yes) (on_board yes) (dnp no) (fields_autoplaced)
-    (property "Reference" "R35" (at 113.03 106.68 0)
+    (property "Reference" "R25" (at 113.03 106.68 0)
       (effects (font (size 1.27 1.27)) (justify right))
     )
@@
     (instances
       (project "av2324"
-        (path "/f5bfae7e-37ef-453c-b315-6458aa70054f"
-          (reference "R35") (unit 1)
-        )
-        (path "/f5bfae7e-37ef-453c-b315-6458aa70054f/32ae0883-da14-4189-aed1-7d6ebb961713"
-          (reference "R35") (unit 1)
-        )
         (path "/f5bfae7e-37ef-453c-b315-6458aa70054f/0748e7cd-0a3d-4586-8bc7-9a3e9814e06f"
           (reference "R25") (unit 1)
@@
   (symbol (lib_id "Device:R_US") (at 127 74.93 0) (unit 1)
     (in_bom yes) (on_board yes) (dnp no) (fields_autoplaced)
-    (property "Reference" "R12" (at 129.54 73.66 0)
+    (property "Reference" "R22" (at 129.54 73.66 0)
       (effects (font (size 1.27 1.27)) (justify left))
     )
@@
     (instances
       (project "av2324"
-        (path "/f5bfae7e-37ef-453c-b315-6458aa70054f"
-          (reference "R12") (unit 1)
-        )
         (path "/f5bfae7e-37ef-453c-b315-6458aa70054f/0748e7cd-0a3d-4586-8bc7-9a3e9814e06f"
           (reference "R22") (unit 1)
